File: kicad_folder/FSAE Club Car (10-19).kicad_sch (KiCad schematic)
At the start: 69 parts, among them J1 ECU PINOUT, J2 ECU PINOUT, J3 ECU PINOUT, J4 Car_Side, J5 Board_Side, K1 Shutdown Relay, K10 starter control relay, K11 starter solenoid, K12 Fans Relay, K13 Shutdown Relay, K14 Main Relay, K15 Fuel pump and Injectors, K16 starter solenoid, K18 starter control relay, K19 Fans Relay, K2 Main Relay, K3 Fuel pump and Injectors, K4 starter control relay, K5 starter solenoid, K6 Fans Relay, K7 Shutdown Relay, K8 Main Relay, K9 Fuel pump and Injectors, SW1 BOTS, SW10 BOTS, SW11 Inertia switch, SW12 Cockpit switch, SW13 starter, SW14 BOTS, SW15 Inertia switch, SW16 Cockpit switch, SW17 starter, SW18 Ignition, SW2 cockpit Switch, SW3 Inertia Switch, SW4 Ignition, SW5 SW_Push, SW9 Ignition

Commit message: separated connectors
Parts:
- added D11, D13, D15, D9: 16V Zener, Package_DIP:DIP-40_W15.24mm, symbol Device:D_Zener
- added D12: D_Zener, Package_DIP:DIP-40_W15.24mm, symbol Device:D_Zener
- added F15: Fans 5A, symbol Device:Fuse
- added F24: O2 heater 10A, symbol Device:Fuse
- added F25: Fuel 5A, symbol Device:Fuse
- added F26: Ignition 5A, symbol Device:Fuse
- added F27: Injector 5A, symbol Device:Fuse
- added F28: Fuse, symbol Device:Fuse
- added J10: ECU PINOUT, symbol Connector_Generic_MountingPin:Conn_01x35_MountingPin
- added J11, _1: Ignition, symbol Connector_Generic:Conn_01x02
- added J12: Ingnition_Coil, symbol Connector_Generic:Conn_01x03
- added J13, _5: MAP, symbol Connector_Generic:Conn_01x03
- added J15, _7: Intake_Air_Temp, symbol Connector_Generic:Conn_01x02
- added J16, J17: Coolant_Sys, symbol Connector_Generic:Conn_01x03
- added J6, _: starter, symbol Connector_Generic:Conn_01x03
- added J7, _2: O2_Sens, symbol Connector_Generic:Conn_01x03
- added J8, _3: FP+INJ, symbol Connector_Generic:Conn_01x03
- added J9, _: Vin+KillSwitches, symbol Connector_Generic:Conn_01x02
- added K17: starter solenoid, Relay_THT:Relay_SPST-NO_Fujitsu_FTR-LYAA005x_FormA_Vertical, symbol Relay:Fujitsu_FTR-LYAA005x
- added K20: starter control relay, Relay_THT:Relay_SPST-NO_Fujitsu_FTR-LYAA005x_FormA_Vertical, symbol Relay:Fujitsu_FTR-LYAA005x
- added K21: Shutdown Relay, Relay_THT:Relay_SPST-NO_Fujitsu_FTR-LYAA005x_FormA_Vertical, symbol Relay:Fujitsu_FTR-LYAA005x
- added K22: Fans Relay, Relay_THT:Relay_SPST-NO_Fujitsu_FTR-LYAA005x_FormA_Vertical, symbol Relay:Fujitsu_FTR-LYAA005x
- added K23: Main Relay, Relay_THT:Relay_SPST-NO_Fujitsu_FTR-LYAA005x_FormA_Vertical, symbol Relay:Fujitsu_FTR-LYAA005x
- added K24: Fuel pump and Injectors, Relay_THT:Relay_SPST-NO_Fujitsu_FTR-LYAA005x_FormA_Vertical, symbol Relay:Fujitsu_FTR-LYAA005x
- added PMS3: SW_SPDT, symbol Switch:SW_SPDT
- added SW19: Ignition, symbol Switch:SW_Push
- added SW20: starter, symbol Switch:SW_Push
- added SW21: BOTS, Button_Switch_SMD:Nidec_Copal_CAS-120A, symbol Switch:SW_Push_Open
- added SW22: Inertia switch, Button_Switch_SMD:Nidec_Copal_CAS-120A, symbol Switch:SW_Push_Open
- added SW23: Cockpit switch, Button_Switch_SMD:Nidec_Copal_CAS-120A, symbol Switch:SW_Push_Open
- added _4: Ignition_Coil, symbol Connector_Generic:Conn_01x03
Connections:
- net +12V: now also PMS3.2 (B)
- net Chassis GND: now also D11.2 (A), D13.2 (A), D9.2 (A), J10.22 (Pin_22), J10.23 (Pin_23), K21.A2, K23.A2
- net GND: now also J10.18 (Pin_18), J15.2 (Pin_2), J17.2 (Pin_2), K22.A1, _2.3 (Pin_3), _4.3 (Pin_3), _5.3 (Pin_3)
- net GNDPWR: now also D12.2 (A), D15.2 (A), K17.A1, K20.A2
- new net: J10.1 (Pin_1), K23.13
- new net: J10.12 (Pin_12), _4.2 (Pin_2)
- new net: D12.1 (K), J10.16 (Pin_16), K22.A2
- new net: J10.24 (Pin_24), _5.1 (Pin_1)
- new net: J10.25 (Pin_25), J17.1 (Pin_1)
- new net: J10.26 (Pin_26), J15.1 (Pin_1)
- new net: J10.28 (Pin_28), _5.2 (Pin_2)
- new net: J10.34 (Pin_34), _2.1 (Pin_1)
- new net: F28.2, J10.8 (Pin_8)
- new net: J10.9 (Pin_9), _3.3 (Pin_3)
- new net: F15.2, J11.1 (Pin_1), K21.13, K23.14, K24.14
- new net: J9.1 (Pin_1), K21.14
- new net: D9.1 (K), J9.2 (Pin_2), K21.A1
- new net: F24.1, _2.2 (Pin_2)
- new net: F24.2, F25.2, F26.2, F27.2, K24.13
- new net: D11.1 (K), J11.2 (Pin_2), K20.13, K23.A1, K24.A1, _.1 (Pin_1)
- new net: K20.14, _.3 (Pin_3)
- new net: D15.1 (K), K20.A1, _.2 (Pin_2)
- new net: J17.3 (Pin_3), K22.14
- new net: F26.1, _4.1 (Pin_1)
- new net: SW19.2, _1.1 (Pin_1)
- new net: SW19.1, _1.2 (Pin_2)
- new net: K17.13, PMS3.3 (C), SW21.1 (A), _.1 (Pin_1)
- new net: SW21.2 (B), SW22.1 (A)
- new net: D13.1 (K), F28.1, K24.A2
- new net: F15.1, K22.13
- new net: J6.3 (Pin_3), K17.A2
- new net: F25.1, _3.1 (Pin_1)
- new net: SW22.2 (B), SW23.1 (A)
- new net: SW23.2 (B), _.2 (Pin_2)
- new net: F27.1, _3.2 (Pin_2)
- new net: J6.2 (Pin_2), SW20.1
- new net: J6.1 (Pin_1), SW20.2
Other:
- note added: "O2_out"
