File: kicad_folder/FSAE Club Car (10-19).kicad_sch (KiCad schematic)
At the start: 111 parts, among them J1 ECU PINOUT, J10 ECU PINOUT, J11 Ignition, J12 Ingnition_Coil, J13 MAP, J15 Intake_Air_Temp, J16 Coolant_Sys, J17 Coolant_Sys, J2 ECU PINOUT, J3 ECU PINOUT, J4 Car_Side, J5 Board_Side, J6 starter, J7 O2_Sens, J8 FP+INJ, J9 Vin+KillSwitches, K1 Shutdown Relay, K10 starter control relay, K11 starter solenoid, K12 Fans Relay, K13 Shutdown Relay, K14 Main Relay, K15 Fuel pump and Injectors, K16 starter solenoid, K17 starter solenoid, K18 starter control relay, K19 Fans Relay, K2 Main Relay, K20 starter control relay, K21 Shutdown Relay, K22 Fans Relay, K23 Main Relay, K24 Fuel pump and Injectors, K3 Fuel pump and Injectors, K4 starter control relay, K5 starter solenoid, K6 Fans Relay, K7 Shutdown Relay, K8 Main Relay, K9 Fuel pump and Injectors, SW1 BOTS, SW10 BOTS, SW11 Inertia switch, SW12 Cockpit switch, SW13 starter, SW14 BOTS, SW15 Inertia switch, SW16 Cockpit switch, SW17 starter, SW18 Ignition, SW19 Ignition, SW2 cockpit Switch, SW20 starter, SW21 BOTS, SW22 Inertia switch, SW23 Cockpit switch, SW3 Inertia Switch, SW4 Ignition, SW5 SW_Push, SW9 Ignition

Commit message: vin
yk what vin is
Parts:
- removed D11, D13, D15, D9: 16V Zener, Package_DIP:DIP-40_W15.24mm, symbol Device:D_Zener
- removed D12: D_Zener, Package_DIP:DIP-40_W15.24mm, symbol Device:D_Zener
- added D12, D13, D15, D16, D17: D, Diode_THT:D_DO-35_SOD27_P7.62mm_Horizontal, symbol Device:D
- added J14: V_in, symbol Connector_Generic:Conn_01x02
- added _6: V_in+, symbol Connector_Generic:Conn_01x02
- J9: value Vin+KillSwitches -> KillSwitches
- _: value Vin+KillSwitches -> Killswitches
Connections:
- net Chassis GND: now also D16.2 (A), D17.2 (A), J14.2 (Pin_2), _6.2 (Pin_2)
- net GND: now also D12.2 (A)
- net GNDPWR: now also D15.2 (A)
- net at J10.16 (Pin_16), K22.A2: now also D12.1 (K)
- net at J9.1 (Pin_1), K21.14: now also J14.1 (Pin_1)
- net at J9.2 (Pin_2), K21.A1: now also D17.1 (K)
- net at J11.2 (Pin_2), K20.13, K23.A1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: now also D13.1 (K), D16.1 (K)
- net at K20.A1, _.2 (Pin_2): now also D15.1 (K)
- net at K17.13, PMS3.3 (C): now also _6.1 (Pin_1); no longer SW21.1 (A), _.1 (Pin_1)
- net at F28.1, K24.A2: now also D13.2 (A)
- new net: SW21.1 (A), _.1 (Pin_1)
Other:
- note added: "+12V_in"
- note added: "Kill_Switches+"
- note added: "Kill_Switches-"

Commit message: stuff
Connections:
- net at D13.1 (K), D16.1 (K), J11.2 (Pin_2)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: no longer K20.13
- net at F15.2, J11.1 (Pin_1), K21.13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: now also K20.13
Other:
- note added: "GND"
Changed lines of the file:
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@@
 		)
 	)
+	(text "GND"
+		(exclude_from_sim no)
+		(at 193.548 501.65 0)
+		(effects
+			(font
+				(size 1.27 1.27)
+			)
+		)
+	)
 	(text "MAP_B"
 		(exclude_from_sim no)
@@
 	)
 	(junction
-		(at 323.85 529.59)
-		(diameter 0)
-		(color 0 0 0 0)
-	)
-	(junction
 		(at 321.31 229.87)
 		(diameter 0)
@@
 	(wire
 		(pts
+			(xy 320.04 534.67) (xy 320.04 532.13)
+		)
+		(stroke
+			(width 0)
+			(type default)
+		)
+	)
+	(wire
+		(pts
 			(xy 300.99 64.77) (xy 300.99 50.8)
 		)
@@
 	(wire
 		(pts
-			(xy 323.85 529.59) (xy 322.58 529.59)
-		)
-		(stroke
-			(width 0)
-			(type default)
-		)
-	)
-	(wire
-		(pts
 			(xy 242.57 342.9) (xy 289.56 342.9)
 		)
@@
 	(wire
 		(pts
+			(xy 320.04 532.13) (xy 349.25 532.13)
+		)
+		(stroke
+			(width 0)
+			(type default)
+		)
+	)
+	(wire
+		(pts
 			(xy 292.1 162.56) (xy 448.31 162.56)
 		)
@@
 	(wire
 		(pts
-			(xy 323.85 529.59) (xy 323.85 534.67)
-		)
-		(stroke
-			(width 0)
-			(type default)
-		)
-	)
-	(wire
-		(pts
 			(xy 711.2 74.93) (xy 713.74 74.93)
 		)
@@
 	(wire
 		(pts
-			(xy 323.85 534.67) (xy 320.04 534.67)
+			(xy 339.09 549.91) (xy 350.52 549.91)
 		)
 		(stroke
@@
 	(wire
 		(pts
-			(xy 339.09 549.91) (xy 350.52 549.91)
+			(xy 311.15 562.61) (xy 311.15 523.24)
 		)
 		(stroke
@@
 	(wire
 		(pts
-			(xy 311.15 562.61) (xy 311.15 523.24)
+			(xy 842.01 57.15) (xy 842.01 59.69)
 		)
 		(stroke
@@
 	(wire
 		(pts
-			(xy 842.01 57.15) (xy 842.01 59.69)
+			(xy 177.8 500.38) (xy 199.39 500.38)
 		)
 		(stroke
@@
 	(wire
 		(pts
-			(xy 177.8 500.38) (xy 199.39 500.38)
+			(xy 416.56 369.57) (xy 389.89 369.57)
 		)
 		(stroke
@@
 	(wire
 		(pts
-			(xy 416.56 369.57) (xy 389.89 369.57)
+			(xy 349.25 502.92) (xy 349.25 509.27)
 		)
 		(stroke
@@
 	(wire
 		(pts
-			(xy 349.25 502.92) (xy 349.25 509.27)
+			(xy 349.25 532.13) (xy 349.25 509.27)
 		)
 		(stroke
@@
 	(wire
 		(pts
-			(xy 351.79 529.59) (xy 323.85 529.59)
+			(xy 322.58 529.59) (xy 351.79 529.59)
 		)
 		(stroke

Commit message: Mystery fuse fix
Parts:
- F28: value Fuse -> 5A ECU fuse
Connections:
- net at D13.2 (A), K24.A2: now also J10.8 (Pin_8); no longer F28.1
- net at J10.1 (Pin_1): now also F28.2; no longer K23.13
- new net: F28.1, K23.13
Changed lines of the file:
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@@
 	(wire
 		(pts
-			(xy 378.46 502.92) (xy 486.41 502.92)
+			(xy 378.46 502.92) (xy 444.5 502.92)
 		)
 		(stroke
@@
 	(wire
 		(pts
+			(xy 452.12 502.92) (xy 486.41 502.92)
+		)
+		(stroke
+			(width 0)
+			(type default)
+		)
+	)
+	(wire
+		(pts
 			(xy 295.91 562.61) (xy 298.45 562.61)
 		)
@@
 	(wire
 		(pts
-			(xy 450.85 520.7) (xy 486.41 520.7)
-		)
-		(stroke
-			(width 0)
-			(type default)
-		)
-	)
-	(wire
-		(pts
 			(xy 248.92 43.18) (xy 248.92 46.99)
 		)
@@
 	(wire
 		(pts
-			(xy 422.91 520.7) (xy 443.23 520.7)
+			(xy 422.91 520.7) (xy 486.41 520.7)
 		)
 		(stroke
@@
 	)
 	(symbol
-		(lib_id "Device:Fuse")
-		(at 447.04 520.7 90)
-		(unit 1)
-		(body_style 1)
-		(exclude_from_sim no)
-		(in_bom yes)
-		(on_board yes)
-		(in_pos_files yes)
-		(dnp no)
-		(fields_autoplaced yes)
-		(property "Reference" "F28"
-			(at 447.04 514.35 90)
-			(show_name no)
-			(do_not_autoplace no)
-			(effects
-				(font
-					(size 1.27 1.27)
-				)
-			)
-		)
-		(property "Value" "Fuse"
-			(at 447.04 516.89 90)
-			(show_name no)
-			(do_not_autoplace no)
-			(effects
-				(font
-					(size 1.27 1.27)
-				)
-			)
-		)
-		(property "Footprint" ""
-			(at 447.04 522.478 90)
-			(hide yes)
-			(show_name no)
-			(do_not_autoplace no)
-			(effects
-				(font
-					(size 1.27 1.27)
-				)
-			)
-		)
-		(property "Datasheet" ""
-			(at 447.04 520.7 0)
-			(hide yes)
-			(show_name no)
-			(do_not_autoplace no)
-			(effects
-				(font
-					(size 1.27 1.27)
-				)
-			)
-		)
-		(property "Description" "Fuse"
-			(at 447.04 520.7 0)
-			(hide yes)
-			(show_name no)
-			(do_not_autoplace no)
-			(effects
-				(font
-					(size 1.27 1.27)
-				)
-			)
-		)
-		(pin "2"
-		)
-		(pin "1"
-		)
-		(instances
-			(project "FSAE Club Car (10-19)"
-				(path "/f4a3be7d-51ca-4426-b777-6c682d495711"
-					(reference "F28")
-					(unit 1)
-				)
-			)
-		)
-	)
-	(symbol
 		(lib_id "power:GNDPWR")
 		(at 665.48 168.91 270)
@@
 					(unit 1)
 				)
+			)
+		)
+	)
+	(symbol
+		(lib_id "Device:Fuse")
+		(at 448.31 502.92 90)
+		(unit 1)
+		(body_style 1)
+		(exclude_from_sim no)
+		(in_bom yes)
+		(on_board yes)
+		(in_pos_files yes)
+		(dnp no)
+		(fields_autoplaced yes)
+		(property "Reference" "F28"
+			(at 448.31 496.57 90)
+			(show_name no)
+			(do_not_autoplace no)
+			(effects
+				(font
+					(size 1.27 1.27)
+				)
+			)
+		)
+		(property "Value" "5A ECU fuse"
+			(at 448.31 499.11 90)
+			(show_name no)
+			(do_not_autoplace no)
+			(effects
+				(font
+					(size 1.27 1.27)
+				)
+			)
+		)
+		(property "Footprint" ""
+			(at 448.31 504.698 90)
+			(hide yes)
+			(show_name no)
+			(do_not_autoplace no)
+			(effects
+				(font
+					(size 1.27 1.27)
+				)
+			)
+		)
+		(property "Datasheet" ""
+			(at 448.31 502.92 0)
+			(hide yes)
+			(show_name no)
+			(do_not_autoplace no)
+			(effects
+				(font
+					(size 1.27 1.27)
+				)
+			)
+		)
+		(property "Description" "Fuse"
+			(at 448.31 502.92 0)
+			(hide yes)
+			(show_name no)
+			(do_not_autoplace no)
+			(effects
+				(font
+					(size 1.27 1.27)
+				)
+			)
+		)
+		(pin "2"
+		)
+		(pin "1"
+		)
+		(instances
+			(project "FSAE Club Car (10-19)"
+				(path "/f4a3be7d-51ca-4426-b777-6c682d495711"
+					(reference "F28")
+					(unit 1)
+				)
